File: hardware/prototype/caligula.kicad_sch (KiCad schematic)
At the start: 102 parts, among them J1 USB2UART, J2 1.47 IPS LCD, J3 ConnBattery, J5 lcd jumper, J6 lcd jumper, J7 lcd jumper, J8 PH Sensor, J9 USB2UART, Q1 SS8050, Q2 SS8050, Q3 SS8050, SW1 RST, SW2 IN1, SW3 Boot, SW4 IN2, SW5 IN4, SW6 IN4, SW7 IN5, U1 CH340C, U10 TL431LP, U11 TPS63002, U2 ESP32-S3-WROOM-1, U3 TPS63001_SEPIC_3V3, U5 BQ24075RGT_DPPM, U6 ADS1115IDGS, U8 OPA2197xD, U9 ICL7660

Commit message: feat: update simulation to use +- 3.6v
Parts:
- removed C30, C32, C33: 10uF, Capacitor_SMD:C_0805_2012Metric_Pad1.18x1.45mm_HandSolder, symbol Device:C
- removed C31: 0.1uF, Capacitor_SMD:C_0805_2012Metric_Pad1.18x1.45mm_HandSolder, symbol Device:C
- removed C9: 100nF, Capacitor_SMD:C_0805_2012Metric_Pad1.18x1.45mm_HandSolder, symbol Device:C
- removed J9: USB2UART, Connector_USB:USB_C_Receptacle_GCT_USB4110, symbol Connector:USB_C_Receptacle_USB2.0_14P
- removed L2: 22uH 1A, Inductor_SMD:L_Bourns_SRP7028A_7.3x6.6mm, symbol Device:L
- removed R33: 20K, Resistor_SMD:R_0805_2012Metric_Pad1.20x1.40mm_HandSolder, symbol Device:R_US
- removed SW7: IN5, Button_Switch_SMD:SW_SPST_Omron_B3FS-100xP, symbol Switch:SW_Push
- removed U10: TL431LP, Package_TO_SOT_THT:TO-92_Inline, symbol Reference_Voltage:TL431LP
- removed U11: TPS63002, Package_SON:Texas_DRC0010J_ThermalVias, symbol Regulator_Switching:TPS63002
- removed U9: ICL7660, symbol Regulator_SwitchedCapacitor:ICL7660
- added C18, C19, C20: 100nF, Capacitor_SMD:C_0805_2012Metric_Pad1.18x1.45mm_HandSolder, symbol Device:C
- added Card1: TF PUSH, easyeda2kicad:TF-SMD_TF-PUSH, symbol easyeda2kicad:TFPUSH
- added J4: USB2UART, Connector_USB:USB_C_Receptacle_GCT_USB4110, symbol Connector:USB_C_Receptacle_USB2.0_14P
- added J9: RTD_PT100, TerminalBlock_Phoenix:TerminalBlock_Phoenix_PT-1,5-3-5.0-H_1x03_P5.00mm_Horizontal, symbol Connector:Screw_Terminal_01x03
- added JP2: 3_OR_2_Wire, Jumper:SolderJumper-3_P1.3mm_Open_RoundedPad1.0x1.5mm, symbol Jumper:SolderJumper_3_Open
- added JP3: 2_Wire, Jumper:SolderJumper-2_P1.3mm_Open_TrianglePad1.0x1.5mm, symbol Jumper:SolderJumper_2_Open
- added R26, R27, R28: 51k, Resistor_SMD:R_0805_2012Metric_Pad1.20x1.40mm_HandSolder, symbol Device:R_US
- added R40: 430 1%, Resistor_SMD:R_0805_2012Metric_Pad1.20x1.40mm_HandSolder, symbol Device:R_US
- added SW7: MST22D18G2, easyeda2kicad:SW-SMD_MST22D18G2, symbol easyeda2kicad:MST22D18G2
- added U4: ICL7660, Package_SO:SOIC-8_3.9x4.9mm_P1.27mm, symbol Regulator_SwitchedCapacitor:ICL7660
- added U7: MAX31865xTP, Package_DFN_QFN:TQFN-20-1EP_5x5mm_P0.65mm_EP3.25x3.25mm, symbol Sensor_Temperature:MAX31865xTP
- added U9: OPA2197xD, Package_SO:SOIC-8_3.9x4.9mm_P1.27mm, symbol Amplifier_Operational:OPA2197xD
- C26, C27: footprint (none) -> Capacitor_SMD:C_0805_2012Metric_Pad1.18x1.45mm_HandSolder
- J3: footprint Connector_PinHeader_2.54mm:PinHeader_1x03_P2.54mm_Vertical -> Connector_JST:JST_XH_S3B-XH-A_1x03_P2.50mm_Horizontal
- R10: value 1k -> 51k
- R32: value 9K -> 1k8
- R34: value 25K -> 10K
- R36: value 100 -> 10K
- SW1, SW3: footprint Button_Switch_SMD:SW_SPST_PTS810 -> Button_Switch_SMD:SW_SPST_EVQP7A
- SW2, SW4, SW5, SW6: footprint Button_Switch_SMD:SW_SPST_Omron_B3FS-100xP -> keyswitches.pretty-master:Kailh_socket_MX_reversible_platemount
Connections:
- net +5V is gone; now on net +3.3V: C25.1, R34.1, U8.8 (V+)
- net +3.3V: now also C18.1, C19.1, Card1.4 (VDD), R26.1, R27.1, R28.1, U4.8 (V+), U7.19 (DVDD), U7.20 (VDD), U9.8 (V+)
- net GND: now also R36.2, C18.2, C19.2, Card1.6 (VSS), J4.A1 (GND), J4.A12 (GND), J4.B1 (GND), J4.B12 (GND), JP2.3 (B), SW7.3, SW7.6, U4.3 (GND), U4.6 (LV), U7.10 (GND), U7.15 (DGND), U7.16 (GND), U7.21 (GND)
- net IN5: no longer R10.2
- net MAX31865CS: now also U2.25 (IO48), U7.13 (~{CS}); no longer U2.17 (IO9)
- net MAX31865DRDY: now also U2.24 (IO47), U7.18 (~{DRDY}); no longer U2.12 (IO8)
- net MISO: now also Card1.7 (DAT0), R26.2
- net MISO2: now also U7.14 (SDO)
- net MOSI: now also R10.2, Card1.3 (CMD)
- net MOSI2: now also U7.11 (SDI)
- net SCK: now also Card1.5 (CLX)
- net SCK2: now also U7.12 (SCLK)
- net VBUS: now also J4.A4 (VBUS), J4.A9 (VBUS), J4.B4 (VBUS), J4.B9 (VBUS)
- net VDD: now also SW7.1, SW7.4; no longer R36.1
- net at R38.2: now also J4.A7 (D-), J4.B7 (D-)
- net at C27.1: now also U4.2 (CAP+)
- net at C27.2: now also U4.4 (CAP-)
- net at R30.2, U8.5 (+): now also R32.1, U8.1
- net at R35.2: now also J4.A5 (CC1)
- net at R39.2: now also J4.A6 (D+), J4.B6 (D+)
- net at C14.1, R15.2, U3.7 (PS/SYNC)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: no longer U3.6 (EN)
- net at R37.2: now also J4.B5 (CC2)
- net +2V5: no longer names the net of R34.2
- net +2V5: now also R36.1, U9.3 (+); no longer R30.1
- net -5V renamed -3V3
- net -3V3: now also U4.5 (VOUT), U9.4 (V-)
- new net: R40.1, U7.1 (BIAS), U7.2 (REFIN+)
- new net: R40.2, U7.3 (REFIN-), U7.4 (ISENSOR)
- new net: J9.3 (Pin_3), JP2.1 (A), JP3.2 (B), U7.5 (FORCE+)
- new net: JP2.2 (C), U7.6 (FORCE2)
- new net: C20.1, J9.2 (Pin_2), JP3.1 (A), U7.7 (RTDIN+)
- new net: C20.2, J9.1 (Pin_1), U7.8 (RTDIN-), U7.9 (FORCE-)
- new net +1.65V: R30.1, U9.1, U9.2 (-)
- new net MMC_CS: Card1.2 (CD/DAT3), R28.2, U2.17 (IO9)
- new net MMC_INT: Card1.8 (DAT1), R27.2, U2.12 (IO8)
- new net TPS_EN: SW7.2, SW7.5, U3.6 (EN)
- no-connect marks 21 -> 24
Other:
- note added: "3 Wire to Force+ 2/4 Wire to GND Connect 2_Wire if use 2/4 Wire"
- note added: "https://github.com/espressif/esp-hosted-mcu/blob/main/docs/sdio.md"
- note added: "https://www.nxp.com/docs/en/application-note/AN2689.pdf"
- note added: "https://www.ti.com/lit/an/snoa529a/snoa529a.pdf"
- note removed: "SEPIC 5V"
- moved on the sheet: C1, C12, C13, C14, C15, C22, C23, C25, C3, C5, C6, D2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

Commit message: chore: tidying up schematic
Parts:
- removed R34, R36: 10K, Resistor_SMD:R_0805_2012Metric_Pad1.20x1.40mm_HandSolder, symbol Device:R_US
- removed U9: OPA2197xD, Package_SO:SOIC-8_3.9x4.9mm_P1.27mm, symbol Amplifier_Operational:OPA2197xD
- added C9: 100nF, Capacitor_SMD:C_0805_2012Metric_Pad1.18x1.45mm_HandSolder, symbol Device:C
- added R33: 10K, Resistor_SMD:R_0805_2012Metric_Pad1.20x1.40mm_HandSolder, symbol Device:R_US
- R32: value 1k8 -> 4k5
Connections:
- net +1.65V is gone; now on net +3.3V: R30.1
- net +3.3V: now also C9.1
- net GND: now also C9.2
- net at R32.1, U8.1: now also R33.1; no longer R30.2, U8.5 (+)
- new net: R30.2, R33.2, U8.5 (+)
Other:
- note added: "+- Converter"
- note added: "ADC"
- note added: "INPUTS"
- note added: "MAX31865"
- note added: "Micro SD"
- note added: "SEPIC ON/OFF"
- moved on the sheet: C1, C10, C11, C12, C13, C14, C15, C16, C17, C18, C19, C2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

Commit message: feat: update component placement
Parts:
- removed J9: RTD_PT100, TerminalBlock_Phoenix:TerminalBlock_Phoenix_PT-1,5-3-5.0-H_1x03_P5.00mm_Horizontal, symbol Connector:Screw_Terminal_01x03
- added J10: PT100_CONN, Connector_Audio:Jack_XLR_Neutrik_NC3FAH1_Horizontal, symbol Connector_Audio:XLR3
Connections:
- net at JP2.1 (A), JP3.2 (B), U7.5 (FORCE+): now also J10.1
- net at C20.1, JP3.1 (A), U7.7 (RTDIN+): now also J10.3
- net at C20.2, U7.8 (RTDIN-), U7.9 (FORCE-): now also J10.2
Other:
- moved on the sheet: C29, J4, R19, R22, R35, R37, R38, R39, SW7, U6

Commit message: feat: update routing phase 1
Connections:
- net GPOUT is gone; now on net IN1: U2.32 (IO39)
- net IN1: no longer U2.33 (IO40)
- net IN2: now also U2.33 (IO40); no longer U2.34 (IO41)
- net IN3: now also U2.34 (IO41); no longer U2.35 (IO42)
- net IN4: now also U2.35 (IO42); no longer U2.26 (IO45)
- net IN5: no longer names the net of U2.16 (IO46)
- no-connect marks 24 -> 26
Changed lines of the file:
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@@
 	)
 	(no_connect
+		(at 209.55 195.58)
+	)
+	(no_connect
 		(at 313.69 274.32)
 	)
@@
 	)
 	(no_connect
+		(at 209.55 198.12)
+	)
+	(no_connect
 		(at 209.55 162.56)
 	)
@@
 	(wire
 		(pts
-			(xy 227.33 195.58) (xy 209.55 195.58)
-		)
-		(stroke
-			(width 0)
-			(type default)
-		)
-	)
-	(wire
-		(pts
 			(xy 293.37 271.78) (xy 288.29 271.78)
 		)
@@
 	(wire
 		(pts
-			(xy 227.33 198.12) (xy 209.55 198.12)
-		)
-		(stroke
-			(width 0)
-			(type default)
-		)
-	)
-	(wire
-		(pts
 			(xy 323.85 264.16) (xy 321.31 264.16)
 		)
@@
 		)
 	)
+	(label "IN3"
+		(at 227.33 190.5 180)
+		(effects
+			(font
+				(size 1.27 1.27)
+			)
+			(justify right bottom)
+		)
+	)
 	(label "EN"
 		(at 175.26 157.48 180)
@@
 		)
 	)
+	(label "IN1"
+		(at 227.33 185.42 180)
+		(effects
+			(font
+				(size 1.27 1.27)
+			)
+			(justify right bottom)
+		)
+	)
 	(label "ADS1115_DRDY"
 		(at 227.33 165.1 180)
@@
 		)
 	)
-	(label "GPOUT"
-		(at 227.33 185.42 180)
+	(label "IN2"
+		(at 227.33 187.96 180)
 		(effects
 			(font
@@
 		)
 	)
-	(label "IN1"
-		(at 227.33 187.96 180)
-		(effects
-			(font
-				(size 1.27 1.27)
-			)
-			(justify right bottom)
-		)
-	)
 	(label "MOSI"
 		(at 422.91 110.49 0)
@@
 		)
 	)
-	(label "IN5"
-		(at 227.33 198.12 180)
-		(effects
-			(font
-				(size 1.27 1.27)
-			)
-			(justify right bottom)
-		)
-	)
 	(label "IN4"
 		(at 234.95 280.67 0)
@@
 		)
 	)
-	(label "IN3"
-		(at 227.33 193.04 180)
-		(effects
-			(font
-				(size 1.27 1.27)
-			)
-			(justify right bottom)
-		)
-	)
 	(label "MMC_CS"
 		(at 422.91 107.95 0)
@@
 		)
 	)
-	(label "IN4"
-		(at 227.33 195.58 180)
+	(label "ILIM"
+		(at 49.53 278.13 0)
 		(effects
 			(font
 				(size 1.27 1.27)
 			)
-			(justify right bottom)
+			(justify left bottom)
 		)
 	)
-	(label "ILIM"
-		(at 49.53 278.13 0)
+	(label "IN4"
+		(at 227.33 193.04 180)
 		(effects
 			(font
 				(size 1.27 1.27)
 			)
-			(justify left bottom)
+			(justify right bottom)
 		)
 	)
@@
 		(effects
 			(font
-				(size 1.27 1.27)
-			)
-			(justify right bottom)
-		)
-	)
-	(label "IN2"
-		(at 227.33 190.5 180)
-		(effects
-			(font

Commit message: feat: rechecking routing
Parts:
- removed J10: PT100_CONN, Connector_Audio:Jack_XLR_Neutrik_NC3FAH1_Horizontal, symbol Connector_Audio:XLR3
- added H5, H6, H7, H8: MountingHole, MountingHole:MountingHole_3.2mm_M3, symbol Mechanical:MountingHole
- added J9: PT100_CONN, Connector_Audio:Jack_XLR_Neutrik_NC3FAH-0_Horizontal, symbol Connector_Audio:XLR3
Connections:
- net at JP2.1 (A), JP3.2 (B), U7.5 (FORCE+): now also J9.1
- net at C20.1, JP3.1 (A), U7.7 (RTDIN+): now also J9.3
- net at C20.2, U7.8 (RTDIN-), U7.9 (FORCE-): now also J9.2
